Commit message: update objects

File: araig_objects/objects/salt.urdf (robot description, URDF)
Before this commit: robot jodsalz, 1 links, 0 joints
Links:
- link base_link: geometry collision box size=0.061 0.046 0.144; visual mesh filename=package://araig_objects/media/models/salt.dae

File: araig_objects/objects/zwieback.urdf (robot description, URDF)
Before this commit: robot zwieback, 1 links, 0 joints
Links:
- link base_link: geometry collision box size=0.142 0.076 0.144; visual mesh filename=package://araig_objects/media/models/zwieback.dae
